File: board/SkyNetV3main.sch (EAGLE design)
At the start: 65 parts, among them IC1 HC_05, IC2 RF4463PRO, IC3 LPC1769, IC4 BCX17, IC5 TPS63001, IC6 MCP73871-2CCI/ML, Q1 32.768KHz, Q2 12MHz, Q3 IRLM6402, Q4 BSS138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

Commit message: pre-molex-connector
Parts:
- added X1: 52745-1290, con-molex:52745-1290
- 1K: value 1k -> 330
- renumbered R3 to 1K
Changed lines of the file:
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@@
 <part name="+3V5" library="supply1" deviceset="+3V3" device=""/>
 <part name="IC4" library="skynet_other" deviceset="BCX17" device=""/>
-<part name="R3" library="rcl" deviceset="R-EU_" device="R0603" value="1k"/>
+<part name="1K" library="rcl" deviceset="R-EU_" device="R0603" value="330"/>
 <part name="+3V9" library="supply1" deviceset="+3V3" device=""/>
 <part name="R4" library="rcl" deviceset="R-EU_" device="R0603" value="1k5"/>
@@
 <part name="B1" library="i7" deviceset="1S" device="" value="PL503465"/>
 <part name="GND8" library="supply1" deviceset="GND" device=""/>
+<part name="X1" library="con-molex" deviceset="52745-1290" device=""/>
 </parts>
 <sheets>
@@
 <instance part="+3V5" gate="G$1" x="215.9" y="172.72"/>
 <instance part="IC4" gate="G$1" x="195.58" y="124.46"/>
-<instance part="R3" gate="G$1" x="187.96" y="111.76" rot="R90"/>
+<instance part="1K" gate="G$1" x="187.96" y="111.76" rot="R90"/>
 <instance part="+3V9" gate="G$1" x="198.12" y="172.72"/>
 <instance part="R4" gate="G$1" x="198.12" y="111.76" rot="R90"/>
@@
 <pinref part="IC3" gate="G$1" pin="P2[9]/USB_CONNECT/RXD2/ENET_MDIO"/>
 <wire x1="160.02" y1="78.74" x2="187.96" y2="78.74" width="0.1524" layer="91"/>
-<pinref part="R3" gate="G$1" pin="1"/>
+<pinref part="1K" gate="G$1" pin="1"/>
 <wire x1="187.96" y1="78.74" x2="187.96" y2="106.68" width="0.1524" layer="91"/>
 </segment>
@@
 <net name="USB-CON-TRANS" class="0">
 <segment>
-<pinref part="R3" gate="G$1" pin="2"/>
+<pinref part="1K" gate="G$1" pin="2"/>
 <wire x1="187.96" y1="116.84" x2="187.96" y2="124.46" width="0.1524" layer="91"/>
 <pinref part="IC4" gate="G$1" pin="B"/>
@@
 <instance part="GND40" gate="1" x="68.58" y="114.3"/>
 <instance part="GND41" gate="1" x="78.74" y="114.3"/>
+<instance part="X1" gate="-1" x="-43.18" y="63.5"/>
+<instance part="X1" gate="-2" x="-43.18" y="60.96"/>
+<instance part="X1" gate="-3" x="-43.18" y="58.42"/>
+<instance part="X1" gate="-4" x="-43.18" y="55.88"/>
+<instance part="X1" gate="-5" x="-43.18" y="53.34"/>
+<instance part="X1" gate="-6" x="-43.18" y="50.8"/>
+<instance part="X1" gate="-7" x="-43.18" y="48.26"/>
+<instance part="X1" gate="-8" x="-43.18" y="45.72"/>
+<instance part="X1" gate="-9" x="-43.18" y="43.18"/>
+<instance part="X1" gate="-10" x="-43.18" y="40.64"/>
+<instance part="X1" gate="-11" x="-43.18" y="38.1"/>
+<instance part="X1" gate="-12" x="-43.18" y="35.56"/>
 </instances>
 <busses>
